File: STM32F103_dev_board.kicad_sch (KiCad schematic)
At the start: 36 parts, among them IC2 FT232RNL-REEL, J1 Conn_ARM_JTAG_SWD_20, J2 Conn_01x20_Pin, J3 Conn_01x20_Pin, J6 USB4800-03-A, U1 STM32F103RBTx, Y1 8MHz, Y2 Crystal_GND23

Commit message: Changed 8MHz oscillator to SMD one
Parts:
- Y1: footprint Crystal:Crystal_HC49-4H_Vertical -> Crystal:Crystal_SMD_HC49-SD_HandSoldering
Changed lines of the file:
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@@
       (effects (font (size 1.27 1.27)) (justify right))
     )
-    (property "Footprint" "Crystal:Crystal_HC49-4H_Vertical" (at 255.27 31.75 0)
+    (property "Footprint" "Crystal:Crystal_SMD_HC49-SD_HandSoldering" (at 255.27 31.75 0)
       (effects (font (size 1.27 1.27)) hide)
     )
